File: pcb/p2000m-cpm-coboard.kicad_sch (KiCad schematic)
At the start: 3 parts, among them J1 EXPANSION BOARD, J2 EXPANSION BOARD, U1 CY62256-70PC

Commit message: Initial commit schematic
Parts:
- added C1, C2, C3, C4, C5, C6: 0.1uF, Capacitor_THT:C_Disc_D5.0mm_W2.5mm_P5.00mm, symbol Device:C_Small
- added C7: 100uF, Capacitor_THT:C_Radial_D6.3mm_H5.0mm_P2.50mm, symbol Device:C_Small
- added J3: T/~{M}, Connector_PinHeader_2.54mm:PinHeader_1x03_P2.54mm_Vertical, symbol Connector:Conn_01x03_Pin
- added J4, J5: POWER, Connector_PinHeader_2.54mm:PinHeader_1x02_P2.54mm_Vertical, symbol Connector:Conn_01x02_Pin
- added R1, R2: 2k2, Resistor_THT:R_Axial_DIN0207_L6.3mm_D2.5mm_P7.62mm_Horizontal, symbol Device:R_Small
- added U2: SST39SF010, Package_DIP:DIP-32_W15.24mm_Socket, symbol Memory_Flash:SST39SF010
- added U3: DIL16, Package_DIP:DIP-16_W7.62mm_Socket, symbol p2000m_components:DIL16
- added U4: 74LS74, Package_DIP:DIP-14_W7.62mm_Socket, symbol 74xx:74LS74
- added U5: 74LS138, Package_DIP:DIP-16_W7.62mm_Socket, symbol 74xx:74LS138
- added U6: 74LS283, Package_DIP:DIP-16_W7.62mm_Socket, symbol 74xx:74LS283
- added U7: 82S123, Package_DIP:DIP-16_W7.62mm_Socket, symbol p2000m_components:82S123
- J1: value EXPANSION BOARD -> CPU BOARD
- U1: footprint Package_DIP:DIP-28_W15.24mm -> Package_DIP:DIP-28_W15.24mm_Socket
Connections:
- net A0: now also U1.10 (A0)
- net A1: now also U1.9 (A1)
- net A10: now also U1.21 (A10)
- net A11: now also U1.23 (A11), U2.12 (A0), U3.10, U7.10 (A0)
- net A12: now also U1.2 (A12), U2.11 (A1), U3.11, U6.5 (A1), U7.11 (A1); no longer J2.23 (Pin_23)
- net A13: now also U1.26 (A13), U2.10 (A2), U3.12, U6.3 (A2), U7.12 (A2); no longer J2.24 (Pin_24)
- net A14: now also U2.9 (A3), U3.13, U6.14 (A3), U7.13 (A3); no longer J2.25 (Pin_25)
- net A2: now also U1.8 (A2)
- net A3: now also U1.7 (A3)
- net A4: now also U1.6 (A4), U5.3 (A2)
- net A5: now also U1.5 (A5), U5.6 (E3)
- net A6: now also U1.4 (A6), U5.2 (A1)
- net A7: now also U1.3 (A7), U5.1 (A0)
- net A8: now also U1.25 (A8)
- net A9: now also U1.24 (A9)
- net D0: now also U1.11 (Q0)
- net D1: now also U1.12 (Q1)
- net D2: now also U1.13 (Q2)
- net D3: now also U1.15 (Q3)
- net D4: now also U1.16 (Q4)
- net D5: now also U1.17 (Q5)
- net D6: now also U1.18 (Q6)
- net D7: now also U1.19 (Q7), U4.2 (D)
- net GND: now also U1.1 (A14), C1.2, C2.2, C3.2, C4.2, C5.2, C6.2, C7.2, J3.1 (Pin_1), J4.2 (Pin_2), J5.2 (Pin_2), U2.16 (GND), U2.2 (A16), U2.23 (A10), U2.25 (A11), U2.26 (A9), U2.27 (A8), U2.28 (A13), U2.29 (A14), U2.3 (A15), U2.4 (A12), U2.5 (A7), U2.6 (A6), U3.8, U4.7 (GND), U5.8 (GND), U6.11 (B4), U6.6 (B1), U6.7 (C0), U6.8 (GND), U7.8 (GND)
- net VCC: now also C1.1, C2.1, C3.1, C4.1, C5.1, C6.1, C7.1, J3.3 (Pin_3), J4.1 (Pin_1), J5.1 (Pin_1), R1.1, R2.1, U2.31 (PGM), U2.32 (VCC), U4.10 (~{S}), U4.11 (C), U4.13 (~{R}), U4.14 (VCC), U4.4 (~{S}), U5.16 (VCC), U6.16 (VCC), U7.16 (VCC)
- net ~{IORQ}: now also U5.4 (E1)
- net ~{RD}: now also U1.22 (~{OE})
- net ~{RES}: now also U4.1 (~{R})
- net ~{WR}: now also U1.27 (~{WE}), U5.5 (E2)
- net D: now reaches J2.2 (Pin_2)
- net D: now also J1.2 (Pin_2)
- net ~{INT}: now reaches J2.29 (Pin_29)
- net ~{INT}: now also J1.29 (Pin_29)
- net ~{WAIT}: now reaches J2.32 (Pin_32)
- net ~{WAIT}: now also J1.32 (Pin_32)
- net ~{M1}: now reaches J2.33 (Pin_33)
- net ~{M1}: now also J1.33 (Pin_33)
- net ~{LOCK}: now reaches J2.35 (Pin_35)
- net ~{LOCK}: now also J1.35 (Pin_35)
- net ~{RFSH}: now reaches J2.36 (Pin_36)
- net ~{RFSH}: now also J1.36 (Pin_36)
- net KBI20: now reaches J2.37 (Pin_37)
- net KBI20: now also J1.37 (Pin_37)
- net ~{PHI}: now reaches J2.38 (Pin_38)
- net ~{PHI}: now also J1.38 (Pin_38)
- net ~{PHI2}: now reaches J2.39 (Pin_39)
- net ~{PHI2}: now also J1.39 (Pin_39)
- net 4MHz: now reaches J2.40 (Pin_40)
- net 4MHz: now also J1.40 (Pin_40)
- net ~{RAMS3}: now reaches U1.20 (~{CS})
- net ~{RAMS3}: now also U2.15 (D2)
- net RAMS2 renamed A15
- net A15: now also U2.8 (A4), U3.14, U7.14 (A4); no longer J2.26 (Pin_26)
- new net: J3.2 (Pin_2), U2.7 (A5)
- new net OUT_$2x: U4.3 (C), U5.15 (O0)
- new net P0: U2.13 (D0), U3.1, U7.1 (O1)
- new net P1: U2.14 (D1), U3.2, U7.2 (O2)
- new net P2: U2.17 (D3), U3.3, U7.3 (O3)
- new net P3: R2.2, U3.4, U7.4 (O4)
- new net P4: R1.2, U3.5, U7.5 (O5)
- new net P5: U2.19 (D5), U3.6, U7.6 (O6)
- new net P6: U2.20 (D6), U3.7, U7.7 (O7)
- new net P7: U2.21 (D7), U3.9, U6.12 (A4), U7.9 (O8)
- new net RA12: J2.23 (Pin_23), U6.4 (S1)
- new net RA13: J2.24 (Pin_24), U6.1 (S2)
- new net RA14: J2.25 (Pin_25), U6.13 (S3)
- new net RA15: J2.26 (Pin_26), U6.10 (S4)
- new net ~{CPM_SEL}: U2.22 (CE), U2.24 (OE), U4.6 (~{Q})
- new net ~{T_SEL}: U4.5 (Q), U6.15 (B3), U6.2 (B2), U7.15 (~{CE})
- no-connect marks 20 -> 16
Other:
- note added: "Manual states D0 (wrong)"
- note added: "P2000 PROM"
- note added: "RAMS1"
- note added: "RAMS2"
- note added: "Select 16 KiB RAM"
- note added: "To CPU board (original PROM socket)"
- note added: "To expansion board"
- note added: "~{CARS1}"
- note added: "~{CARS2}"
- note added: "~{MBEN}"
- note added: "~{ROMS1}"
- note added: "~{ROMS2}"
- note added: "~{VIDS}"
- note removed: "D"
- note removed: "RAM Access Memory 2"
- note removed: "~{INT} ~{IORQ} ~{M1} ~{LOCK} ~{DEW/R2425} PHI2"
- note removed: "~{WAIT} ~{RES} ~{RFSH} PHI T4M"
- title: (none) -> P2000M CP/M Coboard
- moved on the sheet: J2, U1

Commit message: Initial commit of PCB layout and fixing some bugs
Parts:
- removed J5: POWER, Connector_PinHeader_2.54mm:PinHeader_1x02_P2.54mm_Vertical, symbol Connector:Conn_01x02_Pin
- added J5: TERMINAL, TerminalBlock:TerminalBlock_bornier-2_P5.08mm, symbol Connector:Screw_Terminal_01x02
- J1, J2: footprint Connector_PinHeader_2.54mm:PinHeader_2x20_P2.54mm_Vertical -> Connector_IDC:IDC-Header_2x20_P2.54mm_Vertical
Connections:
- net GND: now also J5.1 (Pin_1); no longer U2.6 (A6)
- net VCC: now also J5.2 (Pin_2)
- net ~{MRQ}: now also U2.6 (A6)

Commit message: Polishing PCB
Parts:
- J5: footprint TerminalBlock:TerminalBlock_bornier-2_P5.08mm -> TerminalBlock_RND:TerminalBlock_RND_205-00232_1x02_P5.08mm_Horizontal
Changed lines of the file:
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@@
 			)
 		)
-		(property "Footprint" "TerminalBlock:TerminalBlock_bornier-2_P5.08mm"
+		(property "Footprint" "TerminalBlock_RND:TerminalBlock_RND_205-00232_1x02_P5.08mm_Horizontal"
 			(at 102.87 165.1 0)
 			(hide yes)

Commit message: Adding pull-up resistor to RAMS3/ and updating mappings
Parts:
- added R3: 4k7, Resistor_THT:R_Axial_DIN0207_L6.3mm_D2.5mm_P7.62mm_Horizontal, symbol Device:R_Small
Connections:
- net VCC: now also R3.2
- net ~{RAMS3}: now also R3.1
Changed lines of the file:
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@@
 	(text "Select \n16 KiB RAM"
 		(exclude_from_sim no)
-		(at 212.344 21.59 0)
+		(at 210.566 16.256 0)
 		(effects
 			(font
@@
 	)
 	(junction
+		(at 212.09 22.86)
+		(diameter 0)
+		(color 0 0 0 0)
+	)
+	(junction
 		(at 214.63 31.75)
 		(diameter 0)
@@
 	(wire
 		(pts
+			(xy 212.09 22.86) (xy 212.09 20.32)
+		)
+		(stroke
+			(width 0)
+			(type default)
+		)
+	)
+	(wire
+		(pts
 			(xy 267.97 49.53) (xy 264.16 49.53)
 		)
@@
 	(wire
 		(pts
-			(xy 212.09 36.83) (xy 212.09 30.48)
+			(xy 212.09 36.83) (xy 212.09 22.86)
 		)
 		(stroke
@@
 	(global_label "~{RAMS3}"
 		(shape input)
-		(at 212.09 30.48 90)
+		(at 212.09 20.32 90)
 		(fields_autoplaced yes)
 		(effects
@@
 		)
 		(property "Intersheetrefs" "${INTERSHEET_REFS}"
-			(at 212.09 23.1089 90)
+			(at 212.09 12.9489 90)
 			(hide yes)
 			(show_name no)
@@
 	(symbol
 		(lib_id "power:VCC")
+		(at 207.01 22.86 90)
+		(unit 1)
+		(body_style 1)
+		(exclude_from_sim no)
+		(in_bom yes)
+		(on_board yes)
+		(in_pos_files yes)
+		(dnp no)
+		(fields_autoplaced yes)
+		(property "Reference" "#PWR036"
+			(at 210.82 22.86 0)
+			(hide yes)
+			(show_name no)
+			(do_not_autoplace no)
+			(effects
+				(font
+					(size 1.27 1.27)
+				)
+			)
+		)
+		(property "Value" "VCC"
+			(at 203.2 22.8599 90)
+			(show_name no)
+			(do_not_autoplace no)
+			(effects
+				(font
+					(size 1.27 1.27)
+				)
+				(justify left)
+			)
+		)
+		(property "Footprint" ""
+			(at 207.01 22.86 0)
+			(hide yes)
+			(show_name no)
+			(do_not_autoplace no)
+			(effects
+				(font
+					(size 1.27 1.27)
+				)
+			)
+		)
+		(property "Datasheet" ""
+			(at 207.01 22.86 0)
+			(hide yes)
+			(show_name no)
+			(do_not_autoplace no)
+			(effects
+				(font
+					(size 1.27 1.27)
+				)
+			)
+		)
+		(property "Description" "Power symbol creates a global label with name \"VCC\""
+			(at 207.01 22.86 0)
+			(hide yes)
+			(show_name no)
+			(do_not_autoplace no)
+			(effects
+				(font
+					(size 1.27 1.27)
+				)
+			)
+		)
+		(pin "1"
+		)
+		(instances
+			(project "p2000m-cpm-coboard"
+				(path "/6fd0ac56-88c2-4ff6-8529-422939feb5ef"
+					(reference "#PWR036")
+					(unit 1)
+				)
+			)
+		)
+	)
+	(symbol
+		(lib_id "power:VCC")
 		(at 271.78 140.97 0)
 		(unit 1)
@@
 					(unit 1)
 				)
+			)
+		)
+	)
+	(symbol
+		(lib_id "Device:R_Small")
+		(at 209.55 22.86 270)
+		(unit 1)
+		(body_style 1)
+		(exclude_from_sim no)
+		(in_bom yes)
+		(on_board yes)
+		(in_pos_files yes)
+		(dnp no)
+		(property "Reference" "R3"
+			(at 208.28 24.638 90)
+			(show_name no)
+			(do_not_autoplace no)
+			(effects
+				(font
+					(size 1.016 1.016)
+				)
+				(justify left)
+			)
+		)
+		(property "Value" "4k7"
+			(at 207.772 21.082 90)
+			(show_name no)
+			(do_not_autoplace no)
+			(effects
+				(font
+					(size 1.27 1.27)
+				)
+				(justify left)
+			)
+		)
+		(property "Footprint" "Resistor_THT:R_Axial_DIN0207_L6.3mm_D2.5mm_P7.62mm_Horizontal"
+			(at 209.55 22.86 0)
+			(hide yes)
+			(show_name no)
+			(do_not_autoplace no)
+			(effects
+				(font
+					(size 1.27 1.27)
+				)
+			)
+		)
+		(property "Datasheet" ""
+			(at 209.55 22.86 0)
+			(hide yes)
+			(show_name no)
+			(do_not_autoplace no)
+			(effects
+				(font
+					(size 1.27 1.27)
+				)
+			)
+		)
+		(property "Description" "Resistor, small symbol"
+			(at 209.55 22.86 0)
+			(hide yes)
+			(show_name no)
+			(do_not_autoplace no)
+			(effects
+				(font
+					(size 1.27 1.27)
+				)
+			)
+		)
+		(pin "1"
+		)
+		(pin "2"
+		)
+		(instances
+			(project "p2000m-cpm-coboard"
+				(path "/6fd0ac56-88c2-4ff6-8529-422939feb5ef"
+					(reference "R3")
+					(unit 1)
+				)

Commit message: Replacing DIP for PLCC32 for SST39SF010
Parts:
- U2: footprint Package_DIP:DIP-32_W15.24mm_Socket -> Package_LCC:PLCC-32_THT-Socket
Changed lines of the file:
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@@
 			)
 		)
-		(property "Footprint" "Package_DIP:DIP-32_W15.24mm_Socket"
+		(property "Footprint" "Package_LCC:PLCC-32_THT-Socket"
 			(at 194.31 54.61 0)
 			(hide yes)

Commit message: Adding 82S123 contents
Connections:
- net VCC: now also U4.12 (D)
- no-connect marks 16 -> 15
Other:
- note added: "Manual erroneously mentions D0"
- note removed: "Manual states D0 (wrong)"
Changed lines of the file:
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@@
 		)
 	)
-	(text "Manual states\nD0 (wrong)"
+	(text "Manual erroneously\nmentions D0"
 		(exclude_from_sim no)
 		(at 205.486 118.618 0)
@@
 	)
 	(no_connect
-		(at 38.1 102.87)
-	)
-	(no_connect
 		(at 179.07 77.47)
 	)
@@
 					(unit 1)
 				)
+			)
+		)
+	)
+	(symbol
+		(lib_id "power:VCC")
+		(at 38.1 102.87 90)
+		(unit 1)
+		(body_style 1)
+		(exclude_from_sim no)
+		(in_bom yes)
+		(on_board yes)
+		(in_pos_files yes)
+		(dnp no)
+		(fields_autoplaced yes)
+		(property "Reference" "#PWR037"
+			(at 41.91 102.87 0)
+			(hide yes)
+			(show_name no)
+			(do_not_autoplace no)
+			(effects
+				(font
+					(size 1.27 1.27)
+				)
+			)
+		)
+		(property "Value" "VCC"
+			(at 34.29 102.8699 90)
+			(show_name no)
+			(do_not_autoplace no)
+			(effects
+				(font
+					(size 1.27 1.27)
+				)
+				(justify left)
+			)
+		)
+		(property "Footprint" ""
+			(at 38.1 102.87 0)
+			(hide yes)
+			(show_name no)
+			(do_not_autoplace no)
+			(effects
+				(font
+					(size 1.27 1.27)
+				)
+			)
+		)
+		(property "Datasheet" ""
+			(at 38.1 102.87 0)
+			(hide yes)
+			(show_name no)
+			(do_not_autoplace no)
+			(effects
+				(font
+					(size 1.27 1.27)
+				)
+			)
+		)
+		(property "Description" "Power symbol creates a global label with name \"VCC\""
+			(at 38.1 102.87 0)
+			(hide yes)
+			(show_name no)
+			(do_not_autoplace no)
+			(effects
+				(font
+					(size 1.27 1.27)
+				)
+			)
+		)
+		(pin "1"
+		)
+		(instances
+			(project "p2000m-cpm-coboard"
+				(path "/6fd0ac56-88c2-4ff6-8529-422939feb5ef"
+					(reference "#PWR037")
+					(unit 1)
+				)

Commit message: Rerouting by hand
Parts:
- removed C7: 100uF, Capacitor_THT:C_Radial_D6.3mm_H5.0mm_P2.50mm, symbol Device:C_Small
- added C7: 100uF, Capacitor_THT:CP_Radial_D6.3mm_P2.50mm, symbol Device:C_Polarized
- added C8: 0.1uF, Capacitor_THT:C_Disc_D5.0mm_W2.5mm_P5.00mm, symbol Device:C_Small
- added U8: 74LS02, Package_DIP:DIP-14_W7.62mm_Socket, symbol 74xx:74LS02
Connections:
- net GND: now also U2.6 (A6), C7.2, C8.2, U8.7 (GND)
- net OUT_$2x: now also U8.2, U8.3; no longer U4.3 (C)
- net VCC: now also C7.1, C8.1, U8.11, U8.12, U8.14 (VCC), U8.8, U8.9
- net ~{MRQ}: now also U8.5; no longer U2.6 (A6)
- net ~{RAMS3}: now also U8.6; no longer U1.20 (~{CS})
- new net: U4.3 (C), U8.1
- new net: U1.20 (~{CS}), U8.4
- no-connect marks 15 -> 17
Other:
- moved on the sheet: C1, C5, U1, U3, U4B, U5
