File: pcb/modern-revised/p2000m-cpm-coboard.kicad_sch (KiCad schematic)
At the start: 18 parts, among them J1 CPU BOARD, J2 EXPANSION BOARD, J3 T/~{M}, J4 Atmel-JTAG-10, J5 TERMINAL, U2 CY62128, U3 DIL16, U4 ATF1502AS

Commit message: Redesigning modern board
Parts:
- removed J3: T/~{M}, Connector_PinHeader_2.54mm:PinHeader_1x03_P2.54mm_Vertical, symbol Connector:Conn_01x03_Pin
- removed J4: Atmel-JTAG-10, Connector_IDC:IDC-Header_2x05_P2.54mm_Vertical, symbol atf1504_plcc44_breakout:Atmel-JTAG-10
- J1, J2: footprint Connector_IDC:IDC-Header_2x20_P2.54mm_Vertical -> Connector_PinHeader_2.54mm:PinHeader_2x20_P2.54mm_Vertical
Connections:
- net A11: now also U4.28 (I/O); no longer U4.21 (I/O)
- net A12: now also U4.12 (I/O); no longer U4.41 (I/O/GCLK3)
- net A13: now also U4.16 (I/O); no longer U4.34 (I/O)
- net A14: now also U4.27 (I/O); no longer U4.12 (I/O)
- net A15: now also U4.44 (I/OE1); no longer J1.26 (Pin_26), U4.8 (I/O)
- net A4: now also U4.21 (I/O); no longer U4.14 (I/O)
- net A5: now also U4.24 (I/O); no longer U4.2 (I/OE2/GCLK2)
- net A6: now also U4.25 (I/O/PD2); no longer U4.11 (I/O/PD1)
- net A7: now also U4.26 (I/O); no longer U4.43 (I/GCLK1)
- net D0: now also U4.18 (I/O)
- net D7: now also U4.20 (I/O); no longer U4.19 (I/O)
- net GND: no longer U2.2 (A16), U2.3 (A14), U2.31 (A15)
- net P2: now also U4.41 (I/O/GCLK3); no longer U4.37 (I/O)
- net P3: now also U4.37 (I/O); no longer U4.36 (I/O)
- net P4: now also U4.4 (I/O); no longer U4.33 (I/O)
- net P5: now also U4.36 (I/O); no longer U4.31 (I/O)
- net P6: now also U4.34 (I/O); no longer U4.27 (I/O)
- net P7: now also U4.33 (I/O); no longer U4.28 (I/O)
- net RA12: now also U4.8 (I/O); no longer U4.16 (I/O)
- net RA13: now also U4.6 (I/O); no longer U4.20 (I/O)
- net RA14: now also U4.5 (I/O); no longer U4.17 (I/O)
- net ~{IORQ}: now also U4.2 (I/OE2/GCLK2); no longer U4.6 (I/O)
- net ~{M1}: now also U4.43 (I/GCLK1); no longer U4.4 (I/O)
- net ~{MRQ}: now also U4.31 (I/O); no longer U4.9 (I/O)
- net ~{RAMS3}: now also U4.19 (I/O); no longer U4.29 (I/O)
- net ~{WR}: now also U4.14 (I/O); no longer U4.5 (I/O)
- net RA15 renamed RAMS2_EXP
- net RAMS2_EXP: now also U4.29 (I/O); no longer U4.18 (I/O)
- net TCK: no longer names the net of U4.32 (I/O/TCK)
- net TDI: no longer names the net of U4.7 (I/O/TDI)
- net TDO: no longer names the net of U4.38 (I/O/TDO)
- net TMS: no longer names the net of U4.13 (I/O/TMS)
- new net A14_RAM: U2.3 (A14), U4.11 (I/O/PD1)
- new net A15_RAM: U2.31 (A15), U4.17 (I/O)
- new net A16_RAM: U2.2 (A16), U4.9 (I/O)
- no-connect marks 5 -> 8
